File: low-pass/low-pass.kicad_pcb (KiCad board)
At the start: 4 copper layers, 36 x 16 mm, 10 parts, among them J1 Conn_Coaxial, J2 Conn_Coaxial

Commit message: Added QR code to back
Parts:
- added G***: LOGO, Symbol:qr-lowpass, F.Cu at (135.6, 97.0)
- added G***: LOGO, Symbol:qr-lowpass, F.Cu at (127.6, 84.8)
- added G***: LOGO, Symbol:qr-lowpass, F.Cu at (125.2, 78.2)

Commit message: Slight updates to the layout for possible improvement in isolation of components
Parts:
- removed the G*** at (135.6, 97.0)
- removed the G*** at (127.6, 84.8)
- J1, J2: footprint Connector_Coaxial:SMA_Amphenol_132289_EdgeMount -> Connector_Coaxial:SMA_Samtec_SMA-J-P-H-ST-EM1_EdgeMount
- moved J2 1.20 mm to (143.4, 75.0)
- moved J1 1.15 mm to (118.6, 74.8)
- moved C1 0.20 mm to (122.5, 73.7)
Routing:
- net GND: track 0.00 -> 10.7 mm, vias 14 -> 21
- net Net-(J1-In): track 11.9 -> 10.3 mm
- net Net-(C2-Pad2): track 12.4 -> 13.9 mm
- net Net-(J2-In): track 14.6 -> 15.4 mm
Other:
- board size 36 x 16 mm -> 29 x 16 mm
