File: low-pass/low-pass.kicad_sch (KiCad schematic)
At the start: 13 parts, among them J1 Conn_Coaxial, J2 Conn_Coaxial

Commit message: Slight updates to the layout for possible improvement in isolation of components
Parts:
- J1, J2: footprint Connector_Coaxial:SMA_Amphenol_132289_EdgeMount -> Connector_Coaxial:SMA_Samtec_SMA-J-P-H-ST-EM1_EdgeMount
Changed lines of the file:
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@@
 			)
 		)
-		(property "Footprint" "Connector_Coaxial:SMA_Amphenol_132289_EdgeMount"
+		(property "Footprint" "Connector_Coaxial:SMA_Samtec_SMA-J-P-H-ST-EM1_EdgeMount"
 			(at 102.87 104.14 0)
 			(effects
@@
 			)
 		)
-		(property "Footprint" "Connector_Coaxial:SMA_Amphenol_132289_EdgeMount"
+		(property "Footprint" "Connector_Coaxial:SMA_Samtec_SMA-J-P-H-ST-EM1_EdgeMount"
 			(at 201.93 104.14 0)
 			(effects
